File: trafficlight/trafficlight.kicad_pcb (KiCad board)
At the start: 2 copper layers, 30 x 60 mm, 17 parts, among them J1 Power, U1 LM555xM, U2 4017

Commit message: Update PCB
Parts:
- added G***: LOGO, LOGO, F.Cu at (153.0, 80.6)
- added G***: LOGO, LOGO, F.Cu at (134.0, 99.2)
- C1: value 16uF -> 22uF; footprint Capacitor_SMD:C_0603_1608Metric_Pad1.08x0.95mm_HandSolder -> Capacitor_SMD:C_1206_3216Metric_Pad1.33x1.80mm_HandSolder
- D4, D5, D6, D7: value D -> D_Schottky; footprint Diode_SMD:D_0603_1608Metric_Pad1.05x0.95mm_HandSolder -> Diode_SMD:D_SMA_Handsoldering
- R1: value 18k -> 10k
- R2: value 15k -> 5k
- moved D5 12.4 mm to (131.2, 115.4), turned to -90 degrees
- moved R3 9.04 mm to (135.1, 109.5)
- moved D7 6.84 mm to (138.6, 125.1)
- moved D4 6.55 mm to (138.6, 115.4)
- moved R6 4.60 mm to (134.8, 118.0)
- moved D6 3.18 mm to (131.3, 124.9), turned to 90 degrees
- moved C1 0.74 mm to (152.5, 98.0)
- moved R4 0.55 mm to (135.0, 127.4)
Connections:
- D5 pad 1: Net-(D5-K) -> Net-(D1-A)
- D5 pad 2: Net-(D4-A) -> Net-(D5-A)
- D6 pad 1: Net-(D1-A) -> Net-(D2-A)
- D6 pad 2: Net-(D6-A) -> Net-(D5-A)
- D7 pad 1: Net-(D2-A) -> Net-(D7-K)
- D7 pad 2: Net-(D6-A) -> Net-(D4-A)
- R4 pad 2: Net-(D5-K) -> Net-(D7-K)
- R6 pad 1: Net-(D6-A) -> Net-(D5-A)
- U2 pad 7: Net-(D5-K) -> Net-(D7-K)
Routing:
- net Net-(D5-K): track 27.8 -> 0.00 mm
- net Net-(D7-K): track 0.00 -> 27.4 mm
- net Net-(D5-A): track 0.00 -> 7.19 mm
- net Net-(D1-A): track 47.4 -> 40.3 mm
- net Net-(D4-K): track 17.6 -> 24.5 mm
- net Net-(D6-A): track 4.62 -> 0.00 mm
- net Net-(D4-A): track 16.9 -> 18.6 mm
- net Net-(D2-A): track 38.5 -> 39.9 mm
- net Net-(U1-THR): track 16.8 -> 17.7 mm
Other:
- board text added: "23/3/2025 By B Traffic Light V1"
